File: kicad/_autosave-forrasztos.kicad_sch (KiCad schematic)
At the start: 85 parts, among them J1 24V+-, J2 Conn_01x04_Pin, J3 Conn_01x20_Pin, J4 Conn_01x06_Pin, J5 Conn_01x04_Pin, Q1 AOD409, Q2 MMST2222A, Q3 AOD409, Q4 MMST2222A, SW1 RotaryEncoder_Switch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

Commit message: pcb work
Parts:
- SW2: footprint Button_Switch_SMD:SW_Push_1P1T_NO_CK_PTS125Sx43PSMTR -> (none)
Changed lines of the file:
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@@
       (effects (font (size 1.27 1.27)))
     )
-    (property "Footprint" "Button_Switch_SMD:SW_Push_1P1T_NO_CK_PTS125Sx43PSMTR" (at 204.47 21.59 0)
+    (property "Footprint" "" (at 204.47 21.59 0)
       (effects (font (size 1.27 1.27)) hide)
     )
