File: kicad/forrasztos.kicad_sch (KiCad schematic)
At the start: 85 parts, among them J1 24V+-, J2 Conn_01x04_Pin, J3 Conn_01x20_Pin, J4 Conn_01x06_Pin, J5 Conn_01x04_Pin, Q1 AOD409, Q2 MMST2222A, Q3 AOD409, Q4 MMST2222A, SW1 RotaryEncoder_Switch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

Commit message: redone pcb
Parts:
- added P1: USB_C_Plug_USB2.0, symbol Connector:USB_C_Plug_USB2.0
- J2, J5: footprint Connector_PinHeader_2.54mm:PinHeader_1x04_P2.54mm_Vertical -> Connector_PinHeader_2.54mm:PinHeader_2x04_P2.54mm_Vertical
- SW2: footprint Button_Switch_SMD:SW_Push_1P1T_NO_CK_PTS125Sx43PSMTR -> (none)
Connections:
- net GND: now also P1.A1 (GND), P1.A12 (GND), P1.B1 (GND), P1.B12 (GND), P1.S1 (SHIELD)
- net LCD_CS1: now also U5.18 (PB0); no longer U5.29 (PA8)
- net LCD_CS2: now also U5.19 (PB1); no longer U5.30 (PA9)
- net LCD_DI: now also U5.31 (PA10); no longer U5.33 (PA12)
- net LCD_E: now also U5.29 (PA8); no longer U5.31 (PA10)
- net LCD_RW: now also U5.30 (PA9); no longer U5.32 (PA11)
- net USB_SNS: now reaches U5.38 (PA15)
- new net: P1.A4 (VBUS), P1.A9 (VBUS), P1.B4 (VBUS), P1.B9 (VBUS)
- new net USB_DM: P1.A7 (D-), U5.32 (PA11)
- new net USB_DP: P1.A6 (D+), U5.33 (PA12)
- no-connect marks 3 -> 0
Other:
- moved on the sheet: C22, C9, J2, J5, Q1, Q2, Q3, Q4, R12, R13, R14, R15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
